Commit message: a

File: turtlebot3_description/urdf/turtlebot3_burger.urdf.xacro (robot description, xacro)
@@ -7,5 +7,5 @@
     <parent link="base_footprint"/>
     <child link="base_link"/>
-    <origin xyz="0.0 0.0 0.010" rpy="0 0 0"/>
+    <origin xyz="-0.7 -0.14 0.010" rpy="0 0 -3.1415926"/>
   </joint>
   <link name="base_link">
